File: test1/test1.kicad_sch (KiCad schematic)
At the start: 10 parts, among them U1 LT6238

Commit message: new update
Parts:
- added Input1, Vcc1: Conn_01x02_Pin, Connector_PinHeader_2.00mm:PinHeader_1x02_P2.00mm_Vertical, symbol Connector:Conn_01x02_Pin
- added Screw1, Screw4: MountingHole_Pad, MountingHole:MountingHole_2.2mm_M2_DIN965_Pad_TopBottom, symbol Mechanical:MountingHole_Pad
- Output1: renamed from H1; value MountingHole_Pad -> Conn_01x02_Pin; footprint TestPoint:TestPoint_THTPad_D1.5mm_Drill0.7mm -> Connector_PinHeader_2.00mm:PinHeader_1x02_P2.00mm_Vertical
- Screw2: renamed from H3; footprint TestPoint:TestPoint_THTPad_D1.5mm_Drill0.7mm -> MountingHole:MountingHole_2.2mm_M2_DIN965_Pad_TopBottom
- Screw3: renamed from H2; footprint TestPoint:TestPoint_THTPad_D1.5mm_Drill0.7mm -> MountingHole:MountingHole_2.2mm_M2_DIN965_Pad_TopBottom
- renumbered U1 to uA741
Connections:
- net +5V: now also Vcc1.1 (Pin_1)
- net -5V: now also Vcc1.2 (Pin_2)
- net GND: now also Output1.2 (Input), Screw3.1, Input1.1 (GND), Screw1.1, Screw4.1
- net Input: now reaches R4.2
- net Input: now also Input1.2 (Input); no longer Output1.1
- net Output: now reaches C2.2, R2.1, uA741.6 (OUT)
- net Output: now also Output1.1 (GND); no longer Screw3.1
Other:
- moved on the sheet: Screw2, Screw3
