File: test1/test1.kicad_pcb (KiCad board)
At the start: 2 copper layers, 10 parts, among them U1 LT6238

Commit message: new update
Parts:
- added Input: Conn_01x02_Pin, Connector_PinHeader_2.00mm:PinHeader_1x02_P2.00mm_Vertical, F.Cu at (170.5, 103.0)
- added Screw1: MountingHole_Pad, MountingHole:MountingHole_2.2mm_M2_DIN965_Pad_TopBottom, F.Cu at (128.5, 112.0)
- added Screw4: MountingHole_Pad, MountingHole:MountingHole_2.2mm_M2_DIN965_Pad_TopBottom, F.Cu at (128.5, 89.0)
- added Vcc: Conn_01x02_Pin, Connector_PinHeader_2.00mm:PinHeader_1x02_P2.00mm_Vertical, F.Cu at (151.5, 93.5)
- Output: renamed from H1; value MountingHole_Pad -> Conn_01x02_Pin; footprint TestPoint:TestPoint_THTPad_D1.5mm_Drill0.7mm -> Connector_PinHeader_2.00mm:PinHeader_1x02_P2.00mm_Vertical
- Screw2: renamed from H3; footprint TestPoint:TestPoint_THTPad_D1.5mm_Drill0.7mm -> MountingHole:MountingHole_2.2mm_M2_DIN965_Pad_TopBottom
- Screw3: renamed from H2; footprint TestPoint:TestPoint_THTPad_D1.5mm_Drill0.7mm -> MountingHole:MountingHole_2.2mm_M2_DIN965_Pad_TopBottom
- moved Screw2 76.1 mm to (174.5, 112.0)
- moved Screw3 76.1 mm to (174.5, 89.0)
- moved C2 71.6 mm to (162.5, 104.0)
- moved Output 71.6 mm to (170.5, 98.0)
- moved C1 71.5 mm to (137.5, 104.0)
- moved uA741 71.5 mm to (146.7, 98.2)
- moved R2 70.9 mm to (165.2, 90.0)
- moved R3 70.2 mm to (133.5, 111.0)
- moved R4 70.2 mm to (152.5, 111.0)
- moved R1 69.9 mm to (146.2, 90.0)
- renumbered U1 to uA741
Connections:
- C2 pad 2: Net-(U1-OUT) -> Output
- Output pad 1: Net-(H1-Pad1) -> Output
- R2 pad 1: Net-(U1-OUT) -> Output
- R4 pad 2: Net-(H1-Pad1) -> Input
- Screw3 pad 1: Net-(U1-OUT) -> GND
- uA741 pad 6: Net-(U1-OUT) -> Output
Routing:
- net Net-(U1-OUT): track 36.0 -> 0.00 mm
- net Output: track 0.00 -> 29.4 mm
- net Net-(H1-Pad1): track 22.1 -> 0.00 mm
- net -5V: track 0.00 -> 16.0 mm
- net +5V: track 0.00 -> 12.0 mm
- net Input: track 0.00 -> 10.1 mm
- net Net-(C2-Pad1): track 21.8 -> 19.8 mm
- net Net-(uA741-IN+): track 18.9 -> 18.2 mm
Other:
- board text added: "-Vcc"
- board text added: "C2"
- board text added: "GND"

Commit message: test
Other:
- board outline added: 52 x 29 mm
Changed lines of the file:
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@@
 		(end 177.5 115)
 		(stroke
-			(width 0.2)
-			(type default)
+			(width 0.05)
+			(type solid)
 		)
 		(fill no)
-		(layer "F.Cu")
-		(net 1)
+		(layer "Edge.Cuts")
 	)
 	(gr_text "C2"
